Commit message: Feat: add param to universal_robot version of urdf

File: ur_description/urdf/ur5.urdf.xacro (robot description, xacro)
@@ -67,5 +67,5 @@
     </inertial>
   </xacro:macro>
-  <xacro:macro name="ur5_robot" params="prefix joint_limited
+  <xacro:macro name="ur5_robot" params="prefix joint_limited kinect_on_arm
      shoulder_pan_lower_limit:=${-pi}    shoulder_pan_upper_limit:=${pi}
      shoulder_lift_lower_limit:=${-pi}    shoulder_lift_upper_limit:=${pi}

Commit message: Chore: rm param

File: ur_description/urdf/ur5.urdf.xacro (robot description, xacro)
@@ -67,5 +67,5 @@
     </inertial>
   </xacro:macro>
-  <xacro:macro name="ur5_robot" params="prefix joint_limited kinect_on_arm
+  <xacro:macro name="ur5_robot" params="prefix joint_limited
      shoulder_pan_lower_limit:=${-pi}    shoulder_pan_upper_limit:=${pi}
      shoulder_lift_lower_limit:=${-pi}    shoulder_lift_upper_limit:=${pi}
